Commit message: Added diff_params to control collision radius of wheels; robot model now appears in rviz

File: nuturtle_description/urdf/turtlebot3_burger.urdf.xacro (robot description, xacro)
@@ -2,4 +2,10 @@
 <robot name="turtlebot3_burger" xmlns:xacro="http://ros.org/wiki/xacro">
   <xacro:include filename="$(find nuturtle_description)/urdf/common_properties.xacro"/>
+  <!-- Get properties from arm.yaml configuration -->
+  <xacro:property name="params_yaml_file" value="$(find nuturtle_description)/config/diff_params.yaml"/>
+  <xacro:property name="diff_params" value="${load_yaml(params_yaml_file)}"/>
+  <!-- Properties from arm.yaml -->
+  <xacro:property name="wheel_radius" value="${diff_params['wheel_radius']}"/>
+  <xacro:property name="wheel_track" value="${diff_params['track_width']/2}"/>
   <link name="base_footprint"/>
   <joint name="base_joint" type="fixed">
@@ -33,5 +39,5 @@
     <parent link="base_link"/>
     <child link="wheel_left_link"/>
-    <origin xyz="0.0 0.08 0.023" rpy="-1.57 0 0"/>
+    <origin xyz="0.0 ${wheel_track} 0.023" rpy="-1.57 0 0"/>
     <axis xyz="0 0 1"/>
   </joint>
@@ -47,5 +53,5 @@
       <origin xyz="0 0 0" rpy="0 0 0"/>
       <geometry>
-        <cylinder length="0.018" radius="0.033"/>
+        <cylinder length="0.018" radius="${wheel_radius}"/>
       </geometry>
     </collision>
@@ -61,5 +67,5 @@
     <parent link="base_link"/>
     <child link="wheel_right_link"/>
-    <origin xyz="0.0 -0.080 0.023" rpy="-1.57 0 0"/>
+    <origin xyz="0.0 -${wheel_track} 0.023" rpy="-1.57 0 0"/>
     <axis xyz="0 0 1"/>
   </joint>
@@ -75,5 +81,5 @@
       <origin xyz="0 0 0" rpy="0 0 0"/>
       <geometry>
-        <cylinder length="0.018" radius="0.033"/>
+        <cylinder length="0.018" radius="${wheel_radius}"/>
       </geometry>
     </collision>

Commit message: Added the ability to spawn colorful robots

File: nuturtle_description/urdf/turtlebot3_burger.urdf.xacro (robot description, xacro)
@@ -8,11 +8,12 @@
   <xacro:property name="wheel_radius" value="${diff_params['wheel_radius']}"/>
   <xacro:property name="wheel_track" value="${diff_params['track_width']/2}"/>
-  <link name="base_footprint"/>
-  <joint name="base_joint" type="fixed">
-    <parent link="base_footprint"/>
-    <child link="base_link"/>
+  <xacro:arg name="color" default="black"/>
+  <link name="$(arg color)-base_footprint"/>
+  <joint name="$(arg color)-base_joint" type="fixed">
+    <parent link="$(arg color)-base_footprint"/>
+    <child link="$(arg color)-base_link"/>
     <origin xyz="0.0 0.0 0.010" rpy="0 0 0"/>
   </joint>
-  <link name="base_link">
+  <link name="$(arg color)-base_link">
     <visual>
       <origin xyz="-0.032 0 0.0" rpy="0 0 0"/>
@@ -20,5 +21,5 @@
         <mesh filename="package://nuturtle_description/urdf/meshes/burger_base.stl" scale="0.001 0.001 0.001"/>
       </geometry>
-      <material name="light_black"/>
+      <material name="$(arg color)"/>
     </visual>
     <collision>
@@ -36,11 +37,11 @@
     </inertial>
   </link>
-  <joint name="wheel_left_joint" type="continuous">
-    <parent link="base_link"/>
-    <child link="wheel_left_link"/>
+  <joint name="$(arg color)-wheel_left_joint" type="continuous">
+    <parent link="$(arg color)-base_link"/>
+    <child link="$(arg color)-wheel_left_link"/>
     <origin xyz="0.0 ${wheel_track} 0.023" rpy="-1.57 0 0"/>
     <axis xyz="0 0 1"/>
   </joint>
-  <link name="wheel_left_link">
+  <link name="$(arg color)-wheel_left_link">
     <visual>
       <origin xyz="0 0 0" rpy="1.57 0 0"/>
@@ -64,11 +65,11 @@
       </inertial>
   </link>
-  <joint name="wheel_right_joint" type="continuous">
-    <parent link="base_link"/>
-    <child link="wheel_right_link"/>
+  <joint name="$(arg color)-wheel_right_joint" type="continuous">
+    <parent link="$(arg color)-base_link"/>
+    <child link="$(arg color)-wheel_right_link"/>
     <origin xyz="0.0 -${wheel_track} 0.023" rpy="-1.57 0 0"/>
     <axis xyz="0 0 1"/>
   </joint>
-  <link name="wheel_right_link">
+  <link name="$(arg color)-wheel_right_link">
     <visual>
       <origin xyz="0 0 0" rpy="1.57 0 0"/>
@@ -92,10 +93,10 @@
       </inertial>
   </link>
-  <joint name="caster_back_joint" type="fixed">
-    <parent link="base_link"/>
-    <child link="caster_back_link"/>
+  <joint name="$(arg color)-caster_back_joint" type="fixed">
+    <parent link="$(arg color)-base_link"/>
+    <child link="$(arg color)-caster_back_link"/>
     <origin xyz="-0.081 0 -0.004" rpy="-1.57 0 0"/>
   </joint>
-  <link name="caster_back_link">
+  <link name="$(arg color)-caster_back_link">
     <collision>
       <origin xyz="0 0.001 0" rpy="0 0 0"/>
@@ -112,16 +113,16 @@
     </inertial>
   </link>
-  <joint name="imu_joint" type="fixed">
-    <parent link="base_link"/>
-    <child link="imu_link"/>
+  <joint name="$(arg color)-imu_joint" type="fixed">
+    <parent link="$(arg color)-base_link"/>
+    <child link="$(arg color)-imu_link"/>
     <origin xyz="-0.032 0 0.068" rpy="0 0 0"/>
   </joint>
-  <link name="imu_link"/>
-  <joint name="scan_joint" type="fixed">
-    <parent link="base_link"/>
-    <child link="base_scan"/>
+  <link name="$(arg color)-imu_link"/>
+  <joint name="$(arg color)-scan_joint" type="fixed">
+    <parent link="$(arg color)-base_link"/>
+    <child link="$(arg color)-base_scan"/>
     <origin xyz="-0.032 0 0.172" rpy="0 0 0"/>
   </joint>
-  <link name="base_scan">
+  <link name="$(arg color)-base_scan">
     <visual>
       <origin xyz="0 0 0.0" rpy="0 0 0"/>

Commit message: Added load_all launch file to add four different colored bots to rviz

File: nuturtle_description/urdf/turtlebot3_burger.urdf.xacro (robot description, xacro)
@@ -1,8 +1,8 @@
 <?xml version="1.0" ?>
-<robot name="turtlebot3_burger" xmlns:xacro="http://ros.org/wiki/xacro">
+<robot name="deluxe_burger" xmlns:xacro="http://ros.org/wiki/xacro">
   <xacro:include filename="$(find nuturtle_description)/urdf/common_properties.xacro"/>
   <!-- Get properties from arm.yaml configuration -->
   <xacro:property name="params_yaml_file" value="$(find nuturtle_description)/config/diff_params.yaml"/>
-  <xacro:property name="diff_params" value="${load_yaml(params_yaml_file)}"/>
+  <xacro:property name="diff_params" value="${xacro.load_yaml(params_yaml_file)}"/>
   <!-- Properties from arm.yaml -->
   <xacro:property name="wheel_radius" value="${diff_params['wheel_radius']}"/>

Commit message: Added paramters for collision_radius and motor parameters

File: nuturtle_description/urdf/turtlebot3_burger.urdf.xacro (robot description, xacro)
@@ -2,10 +2,11 @@
 <robot name="deluxe_burger" xmlns:xacro="http://ros.org/wiki/xacro">
   <xacro:include filename="$(find nuturtle_description)/urdf/common_properties.xacro"/>
-  <!-- Get properties from arm.yaml configuration -->
+  <!-- Get properties from diff_params.yaml configuration -->
   <xacro:property name="params_yaml_file" value="$(find nuturtle_description)/config/diff_params.yaml"/>
   <xacro:property name="diff_params" value="${xacro.load_yaml(params_yaml_file)}"/>
-  <!-- Properties from arm.yaml -->
+  <!-- Properties from diff_params.yaml -->
   <xacro:property name="wheel_radius" value="${diff_params['wheel_radius']}"/>
   <xacro:property name="wheel_track" value="${diff_params['track_width']/2}"/>
+  <xacro:property name="collision_radius" value="${diff_params['collision_radius']}"/>
   <xacro:arg name="color" default="black"/>
   <link name="$(arg color)-base_footprint"/>
@@ -26,5 +27,10 @@
       <origin xyz="-0.032 0 0.070" rpy="0 0 0"/>
       <geometry>
-        <box size="0.140 0.140 0.143"/>
+        <xacro:if value="${collision_radius > 0}">
+          <cylinder length="0.143" radius="${collision_radius}"/>
+        </xacro:if>
+        <xacro:unless value="${collision_radius > 0}">
+          <box size="0.140 0.140 0.143"/>
+        </xacro:unless>
       </geometry>
     </collision>
